File: LUNAR-DL.sch (KiCad schematic (older format))
At the start: 1 part

Commit message: Working on schm
Parts:
- removed U?: MAX32625, symbol MAX32625-RESCUE-LUNAR-DL
- added C? (x9): 1uF, symbol C
- added P?: CONN_02X05, symbol CONN_02X05
- added P?: USB_A, symbol USB_A
- added R? (x4): 100K, symbol 1K
- added SW?: SW_PUSH, symbol SW_PUSH
- added U?: MAX32625, symbol MAX32625
- added Y?: Crystal, symbol Crystal
Connections:
- new net: R?.2 (B), SW?.2, U?.21 (RSTN)
- new net: P?.10 (P10), R?.2 (B), U?.22 (SRSTN)
- new net: P?.2 (P2), R?.2 (B), U?.24 (TMS)
- new net: P?.4 (P4), R?.2 (B), U?.26 (TCK)
- new net: U?.35 (32KIN), Y?.2
- new net: U?.36 (32KOUT), Y?.1
- new net: P?.3 (D+), U?.43 (DP)
- new net: P?.2 (D-), U?.44 (DM)
- new net +1V2: C?.1, U?.8 (VDD12)
- new net +1V8: C?.1, C?.1, C?.1, C?.1, C?.1, C?.1, P?.1 (P1), R?.1 (A), R?.1 (A), R?.1 (A), R?.1 (A), U?.23 (VDD18), U?.3 (VDDIO), U?.32 (VDD18), U?.37 (VRTC), U?.42 (VDDIO), U?.46 (VDDIO)
- new net +3V3: C?.1, C?.1, U?.19 (VDDIOH), U?.40 (VDDB)
- new net +5V: P?.1 (VCC)
- new net GND: C?.2, C?.2, C?.2, C?.2, C?.2, C?.2, C?.2, C?.2, C?.2, P?.3 (P3), P?.4 (GND), P?.5 (P5), P?.5 (shield), SW?.1, U?.34 (VSS), U?.41 (VSS), U?.5 (VSS), U?.52 (VSS), U?.63 (VSS)
- new net P2.0_RX: P?.8 (P8), U?.68 (P2.0)
- new net P2.1_TX: P?.6 (P6), U?.67 (P2.1)
